File: r.kicad_sch (KiCad schematic)
At the start: 1 part

Commit message: y not
Parts:
- renumbered R1 to R3
Changed lines of the file:
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@@
   (symbol (lib_id "Device:R") (at 142.875 86.995 0) (unit 1)
     (in_bom yes) (on_board yes) (dnp no) (fields_autoplaced)
-    (property "Reference" "R1" (at 144.78 86.36 0)
+    (property "Reference" "R3" (at 144.78 86.36 0)
       (effects (font (size 1.27 1.27)) (justify left))
     )
@@
       (project "a"
         (path "/63c7d38a-b995-448a-bb92-186d24470b66/34d91a51-52b8-45c3-ad1f-173385eae0c3"
-          (reference "R1") (unit 1)
+          (reference "R3") (unit 1)
         )
       )
