File: r.kicad_sch (KiCad schematic)
At the start: 1 part

Commit message: b again
Parts:
- renumbered R3 to R1
Changed lines of the file:
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@@
   (symbol (lib_id "Device:R") (at 142.875 86.995 0) (unit 1)
     (in_bom yes) (on_board yes) (dnp no) (fields_autoplaced)
-    (property "Reference" "R3" (at 144.78 86.36 0)
+    (property "Reference" "R1" (at 144.78 86.36 0)
       (effects (font (size 1.27 1.27)) (justify left))
     )
@@
       (project "a"
         (path "/63c7d38a-b995-448a-bb92-186d24470b66/34d91a51-52b8-45c3-ad1f-173385eae0c3"
-          (reference "R3") (unit 1)
+          (reference "R1") (unit 1)
         )
       )
+      (project "b"
+        (path "/d97b04af-f940-4b37-9b46-3257568904dc/6b195593-9816-40e7-97c0-c6e7d22a4e06"
+          (reference "R4") (unit 1)
+        )
+      )

Commit message: not this time
Parts:
- renumbered R1 to Rx
Changed lines of the file:
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@@
   (symbol (lib_id "Device:R") (at 142.875 86.995 0) (unit 1)
     (in_bom yes) (on_board yes) (dnp no) (fields_autoplaced)
-    (property "Reference" "R1" (at 144.78 86.36 0)
+    (property "Reference" "Rx" (at 144.78 86.36 0)
       (effects (font (size 1.27 1.27)) (justify left))
     )
@@
       (project "a"
         (path "/63c7d38a-b995-448a-bb92-186d24470b66/34d91a51-52b8-45c3-ad1f-173385eae0c3"
-          (reference "R1") (unit 1)
+          (reference "Rx") (unit 1)
         )
       )

Commit message: another
Parts:
- added Rx1: R, symbol Device:R
Changed lines of the file:
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@@
+    )
+  )
+  (symbol (lib_id "Device:R") (at 154.94 86.995 0) (unit 1)
+    (in_bom yes) (on_board yes) (dnp no) (fields_autoplaced)
+    (property "Reference" "Rx1" (at 157.48 86.36 0)
+      (effects (font (size 1.27 1.27)) (justify left))
+    )
+    (property "Value" "R" (at 157.48 88.9 0)
+      (effects (font (size 1.27 1.27)) (justify left))
+    )
+    (property "Footprint" "" (at 153.162 86.995 90)
+      (effects (font (size 1.27 1.27)) hide)
+    )
+    (property "Datasheet" "~" (at 154.94 86.995 0)
+      (effects (font (size 1.27 1.27)) hide)
+    )
+    (pin "1")
+    (pin "2")
+    (instances
+      (project "a"
+        (path "/63c7d38a-b995-448a-bb92-186d24470b66/34d91a51-52b8-45c3-ad1f-173385eae0c3"
+          (reference "Rx1") (unit 1)
+        )
+      )
+      (project "b"
+        (path "/d97b04af-f940-4b37-9b46-3257568904dc/6b195593-9816-40e7-97c0-c6e7d22a4e06"
+          (reference "R4") (unit 1)
+        )
+      )
     )
   )

Commit message: annot too
Parts:
- renumbered Rx to Rx1, Rx1 to Rx2
Changed lines of the file:
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@@
   (symbol (lib_id "Device:R") (at 142.875 86.995 0) (unit 1)
     (in_bom yes) (on_board yes) (dnp no) (fields_autoplaced)
-    (property "Reference" "Rx" (at 144.78 86.36 0)
+    (property "Reference" "Rx1" (at 144.78 86.36 0)
       (effects (font (size 1.27 1.27)) (justify left))
     )
@@
       (project "a"
         (path "/63c7d38a-b995-448a-bb92-186d24470b66/34d91a51-52b8-45c3-ad1f-173385eae0c3"
-          (reference "Rx") (unit 1)
+          (reference "Rx1") (unit 1)
         )
       )
@@
   (symbol (lib_id "Device:R") (at 154.94 86.995 0) (unit 1)
     (in_bom yes) (on_board yes) (dnp no) (fields_autoplaced)
-    (property "Reference" "Rx1" (at 157.48 86.36 0)
+    (property "Reference" "Rx2" (at 157.48 86.36 0)
       (effects (font (size 1.27 1.27)) (justify left))
     )
@@
       (project "a"
         (path "/63c7d38a-b995-448a-bb92-186d24470b66/34d91a51-52b8-45c3-ad1f-173385eae0c3"
-          (reference "Rx1") (unit 1)
+          (reference "Rx2") (unit 1)
         )
       )
